Commit message: 机器人模型改为匍匐状态的，但是效果不太好，暂存一下

File: tita_description/diablo_plus_pro/urdf/diablo_plus_pro.urdf (robot description, URDF)
Before this commit: robot diablo_pluspro_stand, 8 links, 7 joints
Links:
- removed link imu_link
- link left_wheel_link: mass 2 -> 2.0
- link right_wheel_link: mass 2 -> 2.00
Joints:
- removed joint imu_joint
- joint left_hip_joint: limit lower=-1.57 upper=1.57 effort=80 velocity=15 -> lower=-1.0 upper=1.2 effort=80 velocity=15
- joint left_knee_joint: limit lower=-1.19 upper=0 effort=80 velocity=15 -> lower=0 upper=1.20 effort=80 velocity=15; origin xyz=-0.12022 0.11148 -0.15983 rpy=0 0 0 -> xyz=-0.088027 0.11148 -0.17958 rpy=0 0 0
- joint left_wheel_joint: origin xyz=0.13397 0.01346 -0.1485 rpy=0 0 0 -> xyz=0.17064 0.02266 0.10432 rpy=0 0 0
- joint right_hip_joint: limit lower=-1.57 upper=1.57 effort=80 velocity=15 -> lower=-1.0 upper=1.2 effort=80 velocity=15
- joint right_knee_joint: limit lower=-1.19 upper=0 effort=80 velocity=15 -> lower=0 upper=1.20 effort=80 velocity=15; origin xyz=-0.12022 -0.10364 -0.15983 rpy=0 0 0 -> xyz=-0.088029 -0.10364 -0.17958 rpy=0 0 0
- joint right_wheel_joint: origin xyz=0.13397 -0.03046 -0.1485 rpy=0 0 0 -> xyz=0.17064 -0.03046 0.10432 rpy=0 0 0

File: tita_description/diablo_plus_pro/xacro/description.xacro (robot description, xacro)
@@ -4,5 +4,5 @@
     <link name="base_link">
       <inertial>
-        <origin xyz="0.017899 -0.019179 0.16091" rpy="0 0 0" />
+        <origin xyz="0.02817 -0.0049865 0.16853" rpy="0 0 0" />
         <mass value="8.53" />
         <inertia ixx="0.8371974" ixy="-0.06254957" ixz="-0.01618499" iyy="0.8708397" iyz="0.003006719" izz="0.3425067" />
@@ -11,12 +11,12 @@
         <origin xyz="0 0 0" rpy="0 0 0" />
         <geometry>
-          <mesh filename="file://$(find tita_description)/diablo_pluspro_stand/meshes/base_link.STL" />
-        </geometry>
-        <material name="black"/>
-      </visual>
-      <collision>
-        <origin xyz="0 0 0" rpy="0 0 0" />
-        <geometry>
-          <mesh filename="file://$(find tita_description)/diablo_pluspro_stand/meshes/base_link.STL" />
+          <mesh filename="file://$(find tita_description)/diablo_plus_pro/meshes/base_link.STL" />
+        </geometry>
+        <material name="white"/>
+      </visual>
+      <collision>
+        <origin xyz="0 0 0" rpy="0 0 0" />
+        <geometry>
+          <mesh filename="file://$(find tita_description)/diablo_plus_pro/meshes/base_link.STL" />
         </geometry>
       </collision>
@@ -47,7 +47,7 @@
       <origin rpy="0 0 0" xyz="0 0 0"/>
     </joint>
-    <link name="left_hip_link">
-      <inertial>
-        <origin xyz="-0.028034 0.083955 -0.03225" rpy="0 0 0" />
+   <link name="left_hip_link">
+      <inertial>
+        <origin xyz="-0.02147 0.083955 -0.036946" rpy="0 0 0" />
         <mass value="5.1" />
         <inertia ixx="0.01137421" ixy="0.00070511460" ixz="0.00124554" iyy="0.0082006541" iyz="0.0029798900" izz="0.0060506903" />
@@ -56,12 +56,12 @@
         <origin xyz="0 0 0" rpy="0 0 0" />
         <geometry>
-          <mesh filename="file://$(find tita_description)/diablo_pluspro_stand/meshes/left_hip_link.STL" />
-        </geometry>
-        <material name="black"/>
-      </visual>
-      <collision>
-        <origin xyz="0 0 0" rpy="0 0 0" />
-        <geometry>
-          <mesh filename="file://$(find tita_description)/diablo_pluspro_stand/meshes/left_hip_link.STL" />
+          <mesh filename="file://$(find tita_description)/diablo_plus_pro/meshes/left_hip_link.STL" />
+        </geometry>
+        <material name="white"/>
+      </visual>
+      <collision>
+        <origin xyz="0 0 0" rpy="0 0 0" />
+        <geometry>
+          <mesh filename="file://$(find tita_description)/diablo_plus_pro/meshes/left_hip_link.STL" />
         </geometry>
       </collision>
@@ -72,10 +72,10 @@
       <child link="left_hip_link" />
       <axis xyz="0 1 0" />
-      <limit lower="-1.57" upper="1.57" effort="80" velocity="15" />
+      <limit lower="-1.0" upper="1.2" effort="80" velocity="15" />
     </joint>
     <link name="left_knee_link">
       <inertial>
-        <origin xyz="0.058585 -0.0059746 -0.081982" rpy="0 0 0" />
-        <mass value="2.17" />
+        <origin xyz="0.091371 -0.0059746 0.042483" rpy="0 0 0" />
+        <mass value="2.0" />
         <inertia ixx="0.0044665319" ixy="1.2345077E-05" ixz="-0.00023975799" iyy="0.0046256777" iyz="-0.00022848392" izz="0.0002702575" />
       </inertial>
@@ -83,32 +83,32 @@
         <origin xyz="0 0 0" rpy="0 0 0" />
         <geometry>
-          <mesh filename="file://$(find tita_description)/diablo_pluspro_stand/meshes/left_knee_link.STL" />
-        </geometry>
-        <material name="black"/>
-      </visual>
-      <collision>
-        <origin xyz="0 0 0" rpy="0 0 0" />
-        <geometry>
-          <mesh filename="file://$(find tita_description)/diablo_pluspro_stand/meshes/left_knee_link.STL" />
+          <mesh filename="file://$(find tita_description)/diablo_plus_pro/meshes/left_knee_link.STL" />
+        </geometry>
+        <material name="white"/>
+      </visual>
+      <collision>
+        <origin xyz="0 0 0" rpy="0 0 0" />
+        <geometry>
+          <mesh filename="file://$(find tita_description)/diablo_plus_pro/meshes/left_knee_link.STL" />
         </geometry>
       </collision>
     </link>
     <joint name="left_knee_joint" type="revolute">
-      <origin xyz="-0.12022 0.11148 -0.15983" rpy="0 0 0" />
+      <origin xyz="-0.088027 0.11148 -0.17958" rpy="0 0 0" />
       <parent link="left_hip_link" />
       <child link="left_knee_link" />
       <axis xyz="0 1 0" />
-      <limit lower="-1.19" upper="0" effort="80" velocity="15" />
+      <limit lower="0" upper="1.2" effort="80" velocity="15" />
     </joint>
     <link name="left_wheel_link">
       <inertial>
-        <origin xyz="-2.0554E-06 0.028353 3.331E-07" rpy="0 0 0" />
-        <mass value="2" />
-        <inertia ixx="0.013847" ixy="-1.0976E-07" ixz="-3.0619E-09" iyy="0.027351" iyz="8.9065E-09" izz="0.013847" />
-      </inertial>
-      <visual>
-        <origin xyz="0 0 0" rpy="0 0 0" />
-        <geometry>
-          <mesh filename="file://$(find tita_description)/diablo_pluspro_stand/meshes/left_wheel_link.STL" />
+        <origin xyz="-2.0379E-06 0.019153 -4.2928E-07" rpy="0 0 0" />
+        <mass value="2.0" />
+        <inertia ixx="0.013847" ixy="-1.0562E-07" ixz="4.372E-10" iyy="0.027351" iyz="-3.2677E-08" izz="0.013847" />
+      </inertial>
+      <visual>
+        <origin xyz="0 0 0" rpy="0 0 0" />
+        <geometry>
+          <mesh filename="file://$(find tita_description)/diablo_plus_pro/meshes/left_wheel_link.STL" />
         </geometry>
         <material name="orange"/>
@@ -122,13 +122,13 @@
     </link>
     <joint name="left_wheel_joint" type="revolute">
-      <origin xyz="0.13397 0.01346 -0.1485" rpy="0 0 0" />
+      <origin xyz="0.17064 0.02266 0.10432" rpy="0 0 0" />
       <parent link="left_knee_link" />
       <child link="left_wheel_link" />
       <axis xyz="0 1 0" />
-      <limit lower="-6.283185e4" upper="6.283185e4" effort="20" velocity="30" />
+      <limit lower="-1000000" upper="1000000" effort="20" velocity="30" />
     </joint>
     <link name="right_hip_link">
       <inertial>
-        <origin xyz="-0.028034 -0.083955 -0.032251" rpy="0 0 0" />
+        <origin xyz="-0.02147 -0.083955 -0.036946" rpy="0 0 0" />
         <mass value="5.1" />
         <inertia ixx="0.01137421" ixy="0.00070511460" ixz="0.00124554" iyy="0.0082006541" iyz="0.0029798900" izz="0.0060506903" />
@@ -137,12 +137,12 @@
         <origin xyz="0 0 0" rpy="0 0 0" />
         <geometry>
-          <mesh filename="file://$(find tita_description)/diablo_pluspro_stand/meshes/right_hip_link.STL" />
-        </geometry>
-        <material name="black"/>
-      </visual>
-      <collision>
-        <origin xyz="0 0 0" rpy="0 0 0" />
-        <geometry>
-          <mesh filename="file://$(find tita_description)/diablo_pluspro_stand/meshes/right_hip_link.STL" />
+          <mesh filename="file://$(find tita_description)/diablo_plus_pro/meshes/right_hip_link.STL" />
+        </geometry>
+        <material name="white"/>
+      </visual>
+      <collision>
+        <origin xyz="0 0 0" rpy="0 0 0" />
+        <geometry>
+          <mesh filename="file://$(find tita_description)/diablo_plus_pro/meshes/right_hip_link.STL" />
         </geometry>
       </collision>
@@ -153,9 +153,9 @@
       <child link="right_hip_link" />
       <axis xyz="0 1 0" />
-      <limit lower="-1.57" upper="1.57" effort="80" velocity="15" />
+      <limit lower="-1.0" upper="1.2" effort="80" velocity="15" />
     </joint>
     <link name="right_knee_link">
       <inertial>
-        <origin xyz="0.060903 -0.0019333 -0.083431" rpy="0 0 0" />
+        <origin xyz="0.091173 -0.0018038 0.042402" rpy="0 0 0" />
         <mass value="2.17" />
         <inertia ixx="0.0044665319" ixy="1.2345077E-05" ixz="-0.00023975799" iyy="0.0046256777" iyz="-0.00022848392" izz="0.0002702575" />
@@ -164,32 +164,32 @@
         <origin xyz="0 0 0" rpy="0 0 0" />
         <geometry>
-          <mesh filename="file://$(find tita_description)/diablo_pluspro_stand/meshes/right_knee_link.STL" />
-        </geometry>
-        <material name="black"/>
-      </visual>
-      <collision>
-        <origin xyz="0 0 0" rpy="0 0 0" />
-        <geometry>
-          <mesh filename="file://$(find tita_description)/diablo_pluspro_stand/meshes/right_knee_link.STL" />
+          <mesh filename="file://$(find tita_description)/diablo_plus_pro/meshes/right_knee_link.STL" />
+        </geometry>
+        <material name="white"/>
+      </visual>
+      <collision>
+        <origin xyz="0 0 0" rpy="0 0 0" />
+        <geometry>
+          <mesh filename="file://$(find tita_description)/diablo_plus_pro/meshes/right_knee_link.STL" />
         </geometry>
       </collision>
     </link>
     <joint name="right_knee_joint" type="revolute">
-      <origin xyz="-0.12022 -0.10364 -0.15983" rpy="0 0 0" />
+      <origin xyz="-0.088029 -0.10364 -0.17958" rpy="0 0 0" />
       <parent link="right_hip_link" />
       <child link="right_knee_link" />
       <axis xyz="0 1 0" />
-      <limit lower="-1.19" upper="0" effort="80" velocity="15" />
+      <limit lower="0" upper="1.2" effort="80" velocity="15" />
     </joint>
     <link name="right_wheel_link">
       <inertial>
-        <origin xyz="-2.0311E-06 -0.019153 -4.553E-07" rpy="0 0 0" />
-        <mass value="2" />
-        <inertia ixx="0.013847" ixy="1.0863E-07" ixz="3.5235E-09" iyy="0.027351" iyz="1.5231E-08" izz="0.013847" />
-      </inertial>
-      <visual>
-        <origin xyz="0 0 0" rpy="0 0 0" />
-        <geometry>
-          <mesh filename="file://$(find tita_description)/diablo_pluspro_stand/meshes/right_wheel_link.STL" />
+        <origin xyz="7.6456E-08 -0.019153 -2.0799E-06" rpy="0 0 0" />
+        <mass value="2.0" />
+        <inertia ixx="0.013847" ixy="4.8112E-09" ixz="-1.9773E-09" iyy="0.027351" iyz="1.0933E-07" izz="0.013847" />
+      </inertial>
+      <visual>
+        <origin xyz="0 0 0" rpy="0 0 0" />
+        <geometry>
+          <mesh filename="file://$(find tita_description)/diablo_plus_pro/meshes/right_wheel_link.STL" />
         </geometry>
         <material name="orange"/>
@@ -203,9 +203,9 @@
     </link>
     <joint name="right_wheel_joint" type="revolute">
-      <origin xyz="0.13397 -0.03046 -0.1485" rpy="0 0 0" />
+      <origin xyz="0.17064 -0.03046 0.10432" rpy="0 0 0" />
       <parent link="right_knee_link" />
       <child link="right_wheel_link" />
       <axis xyz="0 1 0" />
-      <limit lower="-6.283185e4" upper="6.283185e4" effort="20" velocity="30" />
+      <limit lower="-1000000" upper="1000000" effort="20" velocity="30" />
     </joint>
   </xacro:macro>

File: tita_description/diablo_plus_pro/xacro/robot.xacro (robot description, xacro)
@@ -6,8 +6,8 @@
   <xacro:property name="ctrl_mode" value="$(arg ctrl_mode)" />
   <xacro:arg name="yaml_path" default="" />
-  <xacro:include filename="$(find tita_description)/diablo_pluspro_stand/xacro/gazebo.xacro" />
-  <xacro:include filename="$(find tita_description)/diablo_pluspro_stand/xacro/materials.xacro" />
-  <xacro:include filename="$(find tita_description)/diablo_pluspro_stand/xacro/description.xacro" />
-  <xacro:include filename="$(find tita_description)/diablo_pluspro_stand/xacro/ros2control.xacro" />
+  <xacro:include filename="$(find tita_description)/diablo_plus_pro/xacro/gazebo.xacro" />
+  <xacro:include filename="$(find tita_description)/diablo_plus_pro/xacro/materials.xacro" />
+  <xacro:include filename="$(find tita_description)/diablo_plus_pro/xacro/description.xacro" />
+  <xacro:include filename="$(find tita_description)/diablo_plus_pro/xacro/ros2control.xacro" />
   <xacro:if value="$(arg use_tower)">
     <xacro:include filename="$(find tita_description)/tower/xacro/tower.urdf.xacro" />

Commit message: 还是切到之前那个分支吧，站着启动感觉也没什么关系好像

File: tita_description/diablo_plus_pro/urdf/diablo_plus_pro.urdf (robot description, URDF)
Before this commit: robot diablo_plus_pro, 7 links, 6 joints
Joints:
- joint left_hip_joint: limit lower=-1.0 upper=1.2 effort=80 velocity=15 -> lower=-1.57 upper=1.57 effort=80 velocity=15
- joint right_hip_joint: limit lower=-1.0 upper=1.2 effort=80 velocity=15 -> lower=-1.57 upper=1.57 effort=80 velocity=15

File: tita_description/diablo_plus_pro/xacro/description.xacro (robot description, xacro)
@@ -72,5 +72,5 @@
       <child link="left_hip_link" />
       <axis xyz="0 1 0" />
-      <limit lower="-1.0" upper="1.2" effort="80" velocity="15" />
+      <limit lower="-1.57" upper="1.57" effort="80" velocity="15" />
     </joint>
     <link name="left_knee_link">
@@ -153,5 +153,5 @@
       <child link="right_hip_link" />
       <axis xyz="0 1 0" />
-      <limit lower="-1.0" upper="1.2" effort="80" velocity="15" />
+      <limit lower="-1.57" upper="1.57" effort="80" velocity="15" />
     </joint>
     <link name="right_knee_link">
