Commit message: 加入了最新导出的质量参数的urdf

File: tita_description/diablo_pluspro/urdf/diablo_pluspro.urdf (robot description, URDF)
Before this commit: robot diablo_pluspro_stand, 8 links, 7 joints
Links:
- removed link imu_link
- link base_link: mass 11.47 -> 16.387
- link left_hip_link: mass 5.1 -> 2.3922754
- link left_knee_link: mass 0.42 -> 0.55812
- link right_hip_link: mass 5.1 -> 2.3922754
- link right_knee_link: mass 0.42 -> 0.55812
Joints:
- removed joint imu_joint
- joint left_hip_joint: limit lower=-1.57 upper=2.0 effort=60 velocity=15 -> lower=-1.57 upper=1.57 effort=60 velocity=15; origin xyz=0 0.0428 0.075997 rpy=0 0 0 -> xyz=0 0.14844 0 rpy=0 0 0
- joint left_knee_joint: origin xyz=-0.12022 0.11148 -0.15983 rpy=0 0 0 -> xyz=-0.12022 0 -0.15983 rpy=0 0 0
- joint left_wheel_joint: origin xyz=0.13397 0.01346 -0.1485 rpy=0 0 0 -> xyz=0.13397 0 -0.1485 rpy=0 0 0
- joint right_hip_joint: limit lower=-1.57 upper=2.0 effort=60 velocity=15 -> lower=-1.57 upper=1.57 effort=60 velocity=15; origin xyz=0 -0.0528 0.075997 rpy=0 0 0 -> xyz=0 -0.1484 0 rpy=0 0 0
- joint right_knee_joint: origin xyz=-0.12022 -0.10364 -0.15983 rpy=0 0 0 -> xyz=-0.12022 0 -0.15983 rpy=0 0 0
- joint right_wheel_joint: origin xyz=0.13397 -0.03046 -0.1485 rpy=0 0 0 -> xyz=0.13397 0 -0.1485 rpy=0 0 0

File: tita_description/diablo_pluspro_stand/xacro/description.xacro (robot description, xacro)
@@ -51,5 +51,10 @@
         <origin xyz="-0.028034 0.083955 -0.03225" rpy="0 0 0" />
         <mass value="5.1" />
-        <inertia ixx="0.01137421" ixy="0.00070511460" ixz="0.00124554" iyy="0.0082006541" iyz="0.0029798900" izz="0.0060506903" />
+        <inertia         ixx="0.052637715"
+        ixy="0.0038396366"
+        ixz="0.0029020553"
+        iyy="0.018328965"
+        iyz="0.0038831563"
+        izz="0.051893499" />
       </inertial>
       <visual>
@@ -72,12 +77,19 @@
       <child link="left_hip_link" />
       <axis xyz="0 1 0" />
-      <limit lower="-1.57" upper="1.57" effort="80" velocity="15" />
+      <dynamics damping="0.6" friction="0.0" />
+      <limit lower="-2.0" upper="2.0" effort="60" velocity="15" />
     </joint>
     <link name="left_knee_link">
       <inertial>
         <origin xyz="0.058585 -0.0059746 -0.081982" rpy="0 0 0" />
-        <mass value="2.17" />
-        <inertia ixx="0.0044665319" ixy="1.2345077E-05" ixz="-0.00023975799" iyy="0.0046256777" iyz="-0.00022848392" izz="0.0002702575" />
-      </inertial>
+        <mass value="0.42" />
+        <inertia
+          ixx="0.0041242120"
+          ixy="-0.00023141797"
+          ixz="-0.0031190064"
+          iyy="0.0068629562"
+          iyz="0.00028573503"
+          izz="0.0028355928" />
+        </inertial>
       <visual>
         <origin xyz="0 0 0" rpy="0 0 0" />
@@ -99,11 +111,18 @@
       <child link="left_knee_link" />
       <axis xyz="0 1 0" />
-      <limit lower="-1.19" upper="0" effort="80" velocity="15" />
+      <dynamics damping="0.6" friction="0.0" />
+      <limit lower="-1.19" upper="0" effort="60" velocity="15" />
     </joint>
     <link name="left_wheel_link">
       <inertial>
         <origin xyz="-2.0554E-06 0.028353 3.331E-07" rpy="0 0 0" />
-        <mass value="2" />
-        <inertia ixx="0.013847" ixy="-1.0976E-07" ixz="-3.0619E-09" iyy="0.027351" iyz="8.9065E-09" izz="0.013847" />
+        <mass value="2.785" />
+        <inertia
+          ixx="0.037393423"
+          ixy="3.1796E-07"
+          ixz="0"
+          iyy="0.073815378"
+          iyz="0"
+          izz="0.037393397" />
       </inertial>
       <visual>
@@ -126,4 +145,5 @@
       <child link="left_wheel_link" />
       <axis xyz="0 1 0" />
+      <dynamics friction="0.01" />
       <limit lower="-6.283185e4" upper="6.283185e4" effort="20" velocity="30" />
     </joint>
@@ -132,5 +152,10 @@
         <origin xyz="-0.028034 -0.083955 -0.032251" rpy="0 0 0" />
         <mass value="5.1" />
-        <inertia ixx="0.01137421" ixy="0.00070511460" ixz="0.00124554" iyy="0.0082006541" iyz="0.0029798900" izz="0.0060506903" />
+        <inertia         ixx="0.052637715"
+        ixy="0.0038396366"
+        ixz="0.0029020553"
+        iyy="0.018328965"
+        iyz="0.0038831563"
+        izz="0.051893499" />
       </inertial>
       <visual>
@@ -153,12 +178,19 @@
       <child link="right_hip_link" />
       <axis xyz="0 1 0" />
-      <limit lower="-1.57" upper="1.57" effort="80" velocity="15" />
+      <dynamics damping="0.6" friction="0.0" />
+      <limit lower="-2.0" upper="2.0" effort="60" velocity="15" />
     </joint>
     <link name="right_knee_link">
       <inertial>
         <origin xyz="0.060903 -0.0019333 -0.083431" rpy="0 0 0" />
-        <mass value="2.17" />
-        <inertia ixx="0.0044665319" ixy="1.2345077E-05" ixz="-0.00023975799" iyy="0.0046256777" iyz="-0.00022848392" izz="0.0002702575" />
-      </inertial>
+        <mass value="0.42" />
+        <inertia
+          ixx="0.0041242120"
+          ixy="-0.00023141797"
+          ixz="-0.0031190064"
+          iyy="0.0068629562"
+          iyz="0.00028573503"
+          izz="0.0028355928" />
+        </inertial>
       <visual>
         <origin xyz="0 0 0" rpy="0 0 0" />
@@ -180,5 +212,6 @@
       <child link="right_knee_link" />
       <axis xyz="0 1 0" />
-      <limit lower="-1.19" upper="0" effort="80" velocity="15" />
+      <dynamics damping="0.6" friction="0.0" />
+      <limit lower="-1.19" upper="0" effort="60" velocity="15" />
     </joint>
     <link name="right_wheel_link">
@@ -186,5 +219,11 @@
         <origin xyz="-2.0311E-06 -0.019153 -4.553E-07" rpy="0 0 0" />
         <mass value="2" />
-        <inertia ixx="0.013847" ixy="1.0863E-07" ixz="3.5235E-09" iyy="0.027351" iyz="1.5231E-08" izz="0.013847" />
+        <inertia
+          ixx="0.037393423"
+          ixy="3.1796E-07"
+          ixz="0"
+          iyy="0.073815378"
+          iyz="0"
+          izz="0.037393397" />
       </inertial>
       <visual>
@@ -207,4 +246,5 @@
       <child link="right_wheel_link" />
       <axis xyz="0 1 0" />
+      <dynamics friction="0.01" />
       <limit lower="-6.283185e4" upper="6.283185e4" effort="20" velocity="30" />
     </joint>
