Commit message: 能平衡了，但是一直会往前走，还要debug一下

File: tita_description/diablo_pluspro_stand/urdf/diablo_pluspro_stand.urdf (robot description, URDF)
Before this commit: robot diablo_pluspro_stand, 8 links, 7 joints
Joints:
- joint left_knee_joint: limit lower=-1.57 upper=0 effort=80 velocity=15 -> lower=-1.19 upper=0 effort=80 velocity=15
- joint right_knee_joint: limit lower=-1.57 upper=0 effort=80 velocity=15 -> lower=-1.19 upper=0 effort=80 velocity=15

File: tita_description/diablo_pluspro_stand/xacro/description.xacro (robot description, xacro)
@@ -99,5 +99,5 @@
       <child link="left_knee_link" />
       <axis xyz="0 1 0" />
-      <limit lower="-1.57" upper="0" effort="80" velocity="15" />
+      <limit lower="-1.19" upper="0" effort="80" velocity="15" />
     </joint>
     <link name="left_wheel_link">
@@ -180,5 +180,5 @@
       <child link="right_knee_link" />
       <axis xyz="0 1 0" />
-      <limit lower="-1.57" upper="0" effort="80" velocity="15" />
+      <limit lower="-1.19" upper="0" effort="80" velocity="15" />
     </joint>
     <link name="right_wheel_link">

Commit message: 尝试修改diablo_pluspro在gazebo中的参数，但是没什么效果；一些limit参数修改

File: tita_description/diablo_pluspro_stand/urdf/diablo_pluspro_stand.urdf (robot description, URDF)
Before this commit: robot diablo_pluspro_stand, 8 links, 7 joints
Joints:
- joint left_wheel_joint: limit effort=20 velocity=30 -> lower=-1000000 upper=1000000 effort=20 velocity=30
- joint right_wheel_joint: limit effort=20 velocity=30 -> lower=-1000000 upper=1000000 effort=20 velocity=30

File: tita_description/diablo_pluspro_stand/xacro/robot.xacro (robot description, xacro)
@@ -6,4 +6,5 @@
   <xacro:property name="ctrl_mode" value="$(arg ctrl_mode)" />
   <xacro:arg name="yaml_path" default="" />
+  <xacro:include filename="$(find tita_description)/diablo_pluspro_stand/xacro/gazebo.xacro" />
   <xacro:include filename="$(find tita_description)/diablo_pluspro_stand/xacro/materials.xacro" />
   <xacro:include filename="$(find tita_description)/diablo_pluspro_stand/xacro/description.xacro" />

Commit message: 修改serial为ttyTHS2，策略更新为适配了新转动惯量的，高度震动变化大

File: tita_description/diablo_pluspro_stand/urdf/diablo_pluspro_stand.urdf (robot description, URDF)
Before this commit: robot diablo_pluspro_stand, 8 links, 7 joints
Links:
- link base_link: mass 8.53 -> 11.47
- link left_knee_link: mass 2.17 -> 0.42
- link right_knee_link: mass 2.17 -> 0.42

File: tita_description/diablo_pluspro_stand/xacro/description.xacro (robot description, xacro)
@@ -5,5 +5,5 @@
       <inertial>
         <origin xyz="0.017899 -0.019179 0.16091" rpy="0 0 0" />
-        <mass value="8.53" />
+        <mass value="11.47" />
         <inertia ixx="0.8371974" ixy="-0.06254957" ixz="-0.01618499" iyy="0.8708397" iyz="0.003006719" izz="0.3425067" />
       </inertial>
@@ -51,5 +51,10 @@
         <origin xyz="-0.028034 0.083955 -0.03225" rpy="0 0 0" />
         <mass value="5.1" />
-        <inertia ixx="0.01137421" ixy="0.00070511460" ixz="0.00124554" iyy="0.0082006541" iyz="0.0029798900" izz="0.0060506903" />
+        <inertia         ixx="0.052637715"
+        ixy="0.0038396366"
+        ixz="0.0029020553"
+        iyy="0.018328965"
+        iyz="0.0038831563"
+        izz="0.051893499" />
       </inertial>
       <visual>
@@ -72,12 +77,19 @@
       <child link="left_hip_link" />
       <axis xyz="0 1 0" />
-      <limit lower="-1.57" upper="1.57" effort="80" velocity="15" />
+      <dynamics damping="1.0" friction="0.0" />
+      <limit lower="-1.57" upper="1.57" effort="60" velocity="15" />
     </joint>
     <link name="left_knee_link">
       <inertial>
         <origin xyz="0.058585 -0.0059746 -0.081982" rpy="0 0 0" />
-        <mass value="2.17" />
-        <inertia ixx="0.0044665319" ixy="1.2345077E-05" ixz="-0.00023975799" iyy="0.0046256777" iyz="-0.00022848392" izz="0.0002702575" />
-      </inertial>
+        <mass value="0.42" />
+        <inertia
+          ixx="0.0041242120"
+          ixy="-0.00023141797"
+          ixz="-0.0031190064"
+          iyy="0.0068629562"
+          iyz="0.00028573503"
+          izz="0.0028355928" />
+        </inertial>
       <visual>
         <origin xyz="0 0 0" rpy="0 0 0" />
@@ -99,5 +111,6 @@
       <child link="left_knee_link" />
       <axis xyz="0 1 0" />
-      <limit lower="-1.19" upper="0" effort="80" velocity="15" />
+      <dynamics damping="1.0" friction="0.0" />
+      <limit lower="-1.19" upper="0" effort="60" velocity="15" />
     </joint>
     <link name="left_wheel_link">
@@ -132,5 +145,10 @@
         <origin xyz="-0.028034 -0.083955 -0.032251" rpy="0 0 0" />
         <mass value="5.1" />
-        <inertia ixx="0.01137421" ixy="0.00070511460" ixz="0.00124554" iyy="0.0082006541" iyz="0.0029798900" izz="0.0060506903" />
+        <inertia         ixx="0.052637715"
+        ixy="0.0038396366"
+        ixz="0.0029020553"
+        iyy="0.018328965"
+        iyz="0.0038831563"
+        izz="0.051893499" />
       </inertial>
       <visual>
@@ -153,12 +171,19 @@
       <child link="right_hip_link" />
       <axis xyz="0 1 0" />
-      <limit lower="-1.57" upper="1.57" effort="80" velocity="15" />
+      <dynamics damping="1.0" friction="0.0" />
+      <limit lower="-1.57" upper="1.57" effort="60" velocity="15" />
     </joint>
     <link name="right_knee_link">
       <inertial>
         <origin xyz="0.060903 -0.0019333 -0.083431" rpy="0 0 0" />
-        <mass value="2.17" />
-        <inertia ixx="0.0044665319" ixy="1.2345077E-05" ixz="-0.00023975799" iyy="0.0046256777" iyz="-0.00022848392" izz="0.0002702575" />
-      </inertial>
+        <mass value="0.42" />
+        <inertia
+          ixx="0.0041242120"
+          ixy="-0.00023141797"
+          ixz="-0.0031190064"
+          iyy="0.0068629562"
+          iyz="0.00028573503"
+          izz="0.0028355928" />
+        </inertial>
       <visual>
         <origin xyz="0 0 0" rpy="0 0 0" />
@@ -180,5 +205,6 @@
       <child link="right_knee_link" />
       <axis xyz="0 1 0" />
-      <limit lower="-1.19" upper="0" effort="80" velocity="15" />
+      <dynamics damping="1.0" friction="0.0" />
+      <limit lower="-1.19" upper="0" effort="60" velocity="15" />
     </joint>
     <link name="right_wheel_link">

Commit message: 准备更新至重新赋值了最新质量与惯量的urdf

File: tita_description/diablo_pluspro_stand/urdf/diablo_pluspro_stand.urdf (robot description, URDF)
Before this commit: robot diablo_pluspro_stand, 8 links, 7 joints
Links:
- link left_wheel_link: mass 2 -> 2.785
- link right_wheel_link: mass 2 -> 2.785
Joints:
- joint left_hip_joint: limit lower=-1.57 upper=1.57 effort=80 velocity=15 -> lower=-1.57 upper=1.57 effort=60 velocity=15
- joint left_knee_joint: limit lower=-1.19 upper=0 effort=80 velocity=15 -> lower=-1.19 upper=0 effort=60 velocity=15
- joint right_hip_joint: limit lower=-1.57 upper=1.57 effort=80 velocity=15 -> lower=-1.57 upper=1.57 effort=60 velocity=15
- joint right_knee_joint: limit lower=-1.19 upper=0 effort=80 velocity=15 -> lower=-1.19 upper=0 effort=60 velocity=15

File: tita_description/diablo_pluspro_stand/xacro/description.xacro (robot description, xacro)
@@ -117,6 +117,12 @@
       <inertial>
         <origin xyz="-2.0554E-06 0.028353 3.331E-07" rpy="0 0 0" />
-        <mass value="2" />
-        <inertia ixx="0.013847" ixy="-1.0976E-07" ixz="-3.0619E-09" iyy="0.027351" iyz="8.9065E-09" izz="0.013847" />
+        <mass value="2.785" />
+        <inertia
+          ixx="0.037393423"
+          ixy="3.1796E-07"
+          ixz="0"
+          iyy="0.073815378"
+          iyz="0"
+          izz="0.037393397" />
       </inertial>
       <visual>
@@ -211,6 +217,12 @@
       <inertial>
         <origin xyz="-2.0311E-06 -0.019153 -4.553E-07" rpy="0 0 0" />
-        <mass value="2" />
-        <inertia ixx="0.013847" ixy="1.0863E-07" ixz="3.5235E-09" iyy="0.027351" iyz="1.5231E-08" izz="0.013847" />
+        <mass value="2.785" />
+        <inertia
+          ixx="0.037393423"
+          ixy="3.1796E-07"
+          ixz="0"
+          iyy="0.073815378"
+          iyz="0"
+          izz="0.037393397" />
       </inertial>
       <visual>
