Commit message: 增大仿真里的关节静摩擦力

File: tita_description/diablo_pluspro/xacro/description.xacro (robot description, xacro)
@@ -74,5 +74,5 @@
       <child link="left_hip_link" />
       <axis xyz="0 1 0" />
-      <dynamics damping="1.0" friction="0.0" />
+      <dynamics damping="0.0" friction="2.0" />
       <limit lower="-3.14" upper="3.14" effort="60" velocity="15" />
     </joint>
@@ -103,5 +103,5 @@
       <child link="left_knee_link" />
       <axis xyz="0 1 0" />
-      <dynamics damping="1.0" friction="0.0" />
+      <dynamics damping="0.0" friction="2.0" />
       <limit lower="-1.19" upper="0" effort="60" velocity="15" />
     </joint>
@@ -161,5 +161,5 @@
       <child link="right_hip_link" />
       <axis xyz="0 1 0" />
-      <dynamics damping="1.0" friction="0.0" />
+      <dynamics damping="0.0" friction="2.0" />
       <limit lower="-3.14" upper="3.14" effort="60" velocity="15" />
     </joint>
@@ -190,5 +190,5 @@
       <child link="right_knee_link" />
       <axis xyz="0 1 0" />
-      <dynamics damping="1.0" friction="0.0" />
+      <dynamics damping="0.0" friction="2.0" />
       <limit lower="-1.19" upper="0" effort="60" velocity="15" />
     </joint>

Commit message: vel range limit

File: tita_description/diablo_pluspro/xacro/description.xacro (robot description, xacro)
@@ -103,5 +103,5 @@
       <child link="left_knee_link" />
       <axis xyz="0 1 0" />
-      <dynamics damping="0.0" friction="2.0" />
+      <dynamics damping="0.0" friction="0.0" />
       <limit lower="-1.19" upper="0" effort="60" velocity="15" />
     </joint>
@@ -110,5 +110,5 @@
       <inertial>
         <origin xyz="0 0.053106868 0" rpy="0 0 0" />
-        <mass value="2.785" />
+        <mass value="4.785" />
         <inertia ixx="0.037393423" ixy="3.1796E-07" ixz="0" iyy="0.073815378" iyz="0" izz="0.037393397" />
       </inertial>
@@ -123,5 +123,5 @@
         <origin xyz="0 0.053 0" rpy="1.5707963 0 0" />
         <geometry>
-          <cylinder radius="0.16" length="0.035"/>
+          <cylinder radius="0.165" length="0.035"/>
         </geometry>
       </collision>
@@ -132,5 +132,5 @@
       <child link="left_wheel_link" />
       <axis xyz="0 1 0" />
-      <dynamics friction="0.01" />
+      <dynamics friction="0" />
       <limit lower="-1000000" upper="1000000" effort="20" velocity="30" />
     </joint>
@@ -190,5 +190,5 @@
       <child link="right_knee_link" />
       <axis xyz="0 1 0" />
-      <dynamics damping="0.0" friction="2.0" />
+      <dynamics damping="0.0" friction="0.0" />
       <limit lower="-1.19" upper="0" effort="60" velocity="15" />
     </joint>
@@ -197,5 +197,5 @@
       <inertial>
         <origin xyz="0 -0.053106868 0" rpy="0 0 0" />
-        <mass value="2.785" />
+        <mass value="4.785" />
         <inertia ixx="0.037393423" ixy="3.1796E-07" ixz="0" iyy="0.073815378" iyz="0" izz="0.037393397" />
       </inertial>
@@ -210,5 +210,5 @@
         <origin xyz="0 -0.053 0" rpy="1.5707963 0 0" />
         <geometry>
-          <cylinder radius="0.16" length="0.035"/>
+          <cylinder radius="0.165" length="0.035"/>
         </geometry>
       </collision>
@@ -219,5 +219,5 @@
       <child link="right_wheel_link" />
       <axis xyz="0 1 0" />
-      <dynamics friction="0.01" />
+      <dynamics friction="0" />
       <limit lower="-1000000" upper="1000000" effort="20" velocity="30" />
     </joint>

File: tita_description/diablo_pluspro/xacro/ros2control.xacro (robot description, xacro)
@@ -86,6 +86,6 @@
         <command_interface name="velocity"/>
         <command_interface name="effort">
-          <param name="min">-80</param>
-          <param name="max">80</param>
+          <param name="min">-60</param>
+          <param name="max">60</param>
         </command_interface>
         <command_interface name="kp"/>
@@ -101,6 +101,6 @@
         <command_interface name="velocity"/>
         <command_interface name="effort">
-          <param name="min">-80</param>
-          <param name="max">80</param>
+          <param name="min">-60</param>
+          <param name="max">60</param>
         </command_interface>
         <command_interface name="kp"/>
@@ -131,6 +131,6 @@
         <command_interface name="velocity"/>
         <command_interface name="effort">
-          <param name="min">-80</param>
-          <param name="max">80</param>
+          <param name="min">-60</param>
+          <param name="max">60</param>
         </command_interface>
         <command_interface name="kp"/>
@@ -146,6 +146,6 @@
         <command_interface name="velocity"/>
         <command_interface name="effort">
-          <param name="min">-80</param>
-          <param name="max">80</param>
+          <param name="min">-60</param>
+          <param name="max">60</param>
         </command_interface>
         <command_interface name="kp"/>

Commit message: 添加mujoco-ros2仿真器

File: tita_description/diablo_pluspro/xacro/description.xacro (robot description, xacro)
@@ -74,5 +74,5 @@
       <child link="left_hip_link" />
       <axis xyz="0 1 0" />
-      <dynamics damping="0.0" friction="2.0" />
+      <dynamics damping="0.0" friction = "0.1" />
       <limit lower="-3.14" upper="3.14" effort="60" velocity="15" />
     </joint>
@@ -103,5 +103,5 @@
       <child link="left_knee_link" />
       <axis xyz="0 1 0" />
-      <dynamics damping="0.0" friction="0.0" />
+      <dynamics damping="0.0" friction = "0.2" />
       <limit lower="-1.19" upper="0" effort="60" velocity="15" />
     </joint>
@@ -110,5 +110,5 @@
       <inertial>
         <origin xyz="0 0.053106868 0" rpy="0 0 0" />
-        <mass value="4.785" />
+        <mass value="2.785" />
         <inertia ixx="0.037393423" ixy="3.1796E-07" ixz="0" iyy="0.073815378" iyz="0" izz="0.037393397" />
       </inertial>
@@ -123,5 +123,5 @@
         <origin xyz="0 0.053 0" rpy="1.5707963 0 0" />
         <geometry>
-          <cylinder radius="0.165" length="0.035"/>
+          <cylinder radius="0.16" length="0.035"/>
         </geometry>
       </collision>
@@ -132,5 +132,5 @@
       <child link="left_wheel_link" />
       <axis xyz="0 1 0" />
-      <dynamics friction="0" />
+      <dynamics damping = "0" friction="0" />
       <limit lower="-1000000" upper="1000000" effort="20" velocity="30" />
     </joint>
@@ -161,5 +161,5 @@
       <child link="right_hip_link" />
       <axis xyz="0 1 0" />
-      <dynamics damping="0.0" friction="2.0" />
+      <dynamics damping="0.0" friction = "0.1" />
       <limit lower="-3.14" upper="3.14" effort="60" velocity="15" />
     </joint>
@@ -190,5 +190,5 @@
       <child link="right_knee_link" />
       <axis xyz="0 1 0" />
-      <dynamics damping="0.0" friction="0.0" />
+      <dynamics damping="0.0" friction = "0.2" />
       <limit lower="-1.19" upper="0" effort="60" velocity="15" />
     </joint>
@@ -197,5 +197,5 @@
       <inertial>
         <origin xyz="0 -0.053106868 0" rpy="0 0 0" />
-        <mass value="4.785" />
+        <mass value="2.785" />
         <inertia ixx="0.037393423" ixy="3.1796E-07" ixz="0" iyy="0.073815378" iyz="0" izz="0.037393397" />
       </inertial>
@@ -210,5 +210,5 @@
         <origin xyz="0 -0.053 0" rpy="1.5707963 0 0" />
         <geometry>
-          <cylinder radius="0.165" length="0.035"/>
+          <cylinder radius="0.16" length="0.035"/>
         </geometry>
       </collision>
@@ -219,5 +219,5 @@
       <child link="right_wheel_link" />
       <axis xyz="0 1 0" />
-      <dynamics friction="0" />
+      <dynamics damping = "0" friction="0" />
       <limit lower="-1000000" upper="1000000" effort="20" velocity="30" />
     </joint>

File: tita_description/diablo_pluspro/xacro/robot.xacro (robot description, xacro)
@@ -28,4 +28,7 @@
     <xacro:property name="name" value="WebotsControl" />
   </xacro:if>
+  <xacro:if value="${sim_env == 'mujoco'}">
+    <xacro:property name="name" value="MujocoControl" />
+  </xacro:if>
   <xacro:description />
   <xacro:ros2control name="${name}" ctrl_mode="$(arg ctrl_mode)" sim_env="$(arg sim_env)" yaml_path="$(arg yaml_path)" />

File: tita_description/diablo_pluspro/xacro/ros2control.xacro (robot description, xacro)
@@ -77,4 +77,7 @@
           <plugin>usr_gazebo_ros2_control/GazeboBridge</plugin>
         </xacro:if>
+        <xacro:if value="${sim_env == 'mujoco'}">
+          <plugin>mujoco_ros2_control/MujocoBridge</plugin>
+        </xacro:if>
         <xacro:if value="${sim_env == 'none'}">
           <plugin>tita_locomotion::HardwareBridge</plugin>
@@ -92,5 +95,5 @@
         <command_interface name="kd"/>
         <state_interface name="position">
-          <param name="initial_value">0.0</param>
+          <param name="initial_value">-0.19</param>
         </state_interface>
         <state_interface name="velocity"/>
@@ -107,5 +110,5 @@
         <command_interface name="kd"/>
         <state_interface name="position">
-          <param name="initial_value">0.0</param>
+          <param name="initial_value">-1.19</param>
         </state_interface>
         <state_interface name="velocity"/>
@@ -137,5 +140,5 @@
         <command_interface name="kd"/>
         <state_interface name="position">
-          <param name="initial_value">0.0</param>
+          <param name="initial_value">-0.19</param>
         </state_interface>
         <state_interface name="velocity"/>
@@ -152,5 +155,5 @@
         <command_interface name="kd"/>
         <state_interface name="position">
-          <param name="initial_value">0.0</param>
+          <param name="initial_value">-1.19</param>
         </state_interface>
         <state_interface name="velocity"/>
