Commit message: 准备迁到单独的分支来部署ddt_b1

File: tita_description/ddt_b1/xacro/materials.xacro (robot description, xacro)
@@ -1,15 +1,30 @@
 <?xml version="1.0"?>
-<robot xmlns:xacro="http://www.ros.org/wiki/xacro">
-  <material name="red">
-    <color rgba="1.0 0.0 0.0 1.0"/>
+<robot>
+  <material name="black">
+    <color rgba="${50/255} ${50/255} ${50/255} 1.0" />
+  </material>
+  <material name="blue">
+    <color rgba="0.0 0.0 0.8 1.0" />
+  </material>
+  <material name="green">
+    <color rgba="0.0 0.8 0.0 1.0" />
+  </material>
+  <material name="grey">
+    <color rgba="0.2 0.2 0.2 1.0" />
   </material>
   <material name="silver">
-    <color rgba="0.75294 0.75294 0.75294 1.0"/>
+    <color rgba="${233/255} ${233/255} ${216/255} 1.0" />
   </material>
-  <material name="grey">
-    <color rgba="0.69804 0.69804 0.69804 1.0"/>
+  <material name="orange">
+    <color rgba="${255/255} ${108/255} ${10/255} 1.0" />
+  </material>
+  <material name="brown">
+    <color rgba="${222/255} ${207/255} ${195/255} 1.0" />
+  </material>
+  <material name="red">
+    <color rgba="0.8 0.0 0.0 1.0" />
   </material>
   <material name="white">
-    <color rgba="1.0 1.0 1.0 1.0"/>
+    <color rgba="1.0 1.0 1.0 1.0" />
   </material>
 </robot>
