Commit message: 加入ddt_b1的相关控制器配置，已能在gazebo中正确显示机器人

File: tita_description/ddt_b1/xacro/description.xacro (robot description, xacro)
@@ -72,5 +72,5 @@
         <origin rpy="0 0 0" xyz="0 0 0"/>
         <geometry>
-          <mesh filename="package://tita_description/ddt_b1/meshes/base_link.STL"/>
+          <mesh filename="file://$(find tita_description)/ddt_b1/meshes/base_link.STL"/>
         </geometry>
         <material name="silver"/>
@@ -104,5 +104,5 @@
         <origin rpy="0 0 0" xyz="0 0 0"/>
         <geometry>
-          <mesh filename="package://tita_description/ddt_b1/meshes/L_hip.STL"/>
+          <mesh filename="file://$(find tita_description)/ddt_b1/meshes/L_hip.STL"/>
         </geometry>
         <material name="silver"/>
@@ -127,5 +127,5 @@
         <origin rpy="0 0 0" xyz="0 0 0"/>
         <geometry>
-          <mesh filename="package://tita_description/ddt_b1/meshes/L_thigh.STL"/>
+          <mesh filename="file://$(find tita_description)/ddt_b1/meshes/L_thigh.STL"/>
         </geometry>
         <material name="silver"/>
@@ -156,5 +156,5 @@
         <origin rpy="0 0 0" xyz="0 0 0"/>
         <geometry>
-          <mesh filename="package://tita_description/ddt_b1/meshes/L_calf.STL"/>
+          <mesh filename="file://$(find tita_description)/ddt_b1/meshes/L_calf.STL"/>
         </geometry>
         <material name="silver"/>
@@ -185,7 +185,7 @@
         <origin rpy="0 0 0" xyz="0 0 0"/>
         <geometry>
-          <mesh filename="package://tita_description/ddt_b1/meshes/L_foot.STL"/>
-        </geometry>
-        <material name="grey"/>
+          <mesh filename="file://$(find tita_description)/ddt_b1/meshes/L_foot.STL"/>
+        </geometry>
+        <material name="black"/>
       </visual>
       <collision>
@@ -214,5 +214,5 @@
         <origin rpy="0 0 0" xyz="0 0 0"/>
         <geometry>
-          <mesh filename="package://tita_description/ddt_b1/meshes/R_hip.STL"/>
+          <mesh filename="file://$(find tita_description)/ddt_b1/meshes/R_hip.STL"/>
         </geometry>
         <material name="silver"/>
@@ -237,5 +237,5 @@
         <origin rpy="0 0 0" xyz="0 0 0"/>
         <geometry>
-          <mesh filename="package://tita_description/ddt_b1/meshes/R_thigh.STL"/>
+          <mesh filename="file://$(find tita_description)/ddt_b1/meshes/R_thigh.STL"/>
         </geometry>
         <material name="silver"/>
@@ -266,5 +266,5 @@
         <origin rpy="0 0 0" xyz="0 0 0"/>
         <geometry>
-          <mesh filename="package://tita_description/ddt_b1/meshes/R_calf.STL"/>
+          <mesh filename="file://$(find tita_description)/ddt_b1/meshes/R_calf.STL"/>
         </geometry>
         <material name="silver"/>
@@ -295,7 +295,7 @@
         <origin rpy="0 0 0" xyz="0 0 0"/>
         <geometry>
-          <mesh filename="package://tita_description/ddt_b1/meshes/R_foot.STL"/>
-        </geometry>
-        <material name="white"/>
+          <mesh filename="file://$(find tita_description)/ddt_b1/meshes/R_foot.STL"/>
+        </geometry>
+        <material name="black"/>
       </visual>
       <collision>

File: tita_description/ddt_b1/xacro/gazebo.xacro (robot description, xacro)
@@ -5,5 +5,5 @@
     <!-- ================================================================== -->
     <!-- IMU Settings -->
-    <xacro:property name="imu_update_rate" value="400.0"/>
+    <xacro:property name="imu_update_rate" value="500.0"/>
     <!-- Leg Link Friction (Hip, Thigh, Calf) -->
     <xacro:property name="leg_mu1" value="0.2"/>
@@ -19,10 +19,4 @@
     <!--                         Gazebo Plugins                             -->
     <!-- ================================================================== -->
-    <!-- ROS2 Control Plugin -->
-    <gazebo>
-      <plugin filename="libgazebo_ros2_control.so" name="gazebo_ros2_control">
-        <parameters>$(arg yaml_path)</parameters>
-      </plugin>
-    </gazebo>
     <!-- IMU Plugin -->
     <gazebo reference="imu_link">

File: tita_description/ddt_b1/xacro/robot.xacro (robot description, xacro)
@@ -2,9 +2,7 @@
 <robot xmlns:xacro="http://wiki.ros.org/xacro" name="ddt_b1">
   <xacro:arg name="prefix" default="" />
-  <xacro:arg name="sim_env" default="none" />
-  <xacro:arg name="ctrl_mode" default="effort" />
-  <xacro:arg name="yaml_path" default="" />
   <xacro:property name="sim_env" value="$(arg sim_env)" />
   <xacro:property name="ctrl_mode" value="$(arg ctrl_mode)" />
+  <xacro:arg name="yaml_path" default="" />
   <xacro:include filename="$(find tita_description)/ddt_b1/xacro/gazebo.xacro" />
   <xacro:include filename="$(find tita_description)/ddt_b1/xacro/materials.xacro" />

File: tita_description/ddt_b1/xacro/ros2control.xacro (robot description, xacro)
@@ -31,10 +31,29 @@
     <!-- ================================================================== -->
     <xacro:if value="${sim_env == 'gazebo'}">
+      <gazebo reference="imu_link">
+        <gravity>true</gravity>
+        <sensor name="imu" type="imu">
+          <always_on>true</always_on>
+          <update_rate>500</update_rate>
+          <!-- <visualize>true</visualize>
+            <topic>__default_topic__</topic>
+            <plugin filename="libgazebo_ros_imu_sensor.so" name="imu_plugin">
+                <topicName>base_imu</topicName>
+                <bodyName>imu_link</bodyName>
+                <updateRateHZ>1000.0</updateRateHZ>
+                <gaussianNoise>0.00</gaussianNoise>
+                <xyzOffset>0 0 0</xyzOffset>
+                <rpyOffset>0 0 0</rpyOffset>
+                <frameName>imu_link</frameName>
+            </plugin>
+            <pose>0 0 0 0 0 0</pose> -->
+        </sensor>
+      </gazebo>
       <gazebo reference="base_link">
         <gravity>true</gravity>
       </gazebo>
       <gazebo reference="F_base_link">
-        <gravity>true</gravity>
         <self_collide>false</self_collide>
+        <gravity>true</gravity>
       </gazebo>
       <!-- Left Leg Gravity -->
@@ -217,5 +236,5 @@
       </joint>
       <!-- IMU Sensor -->
-      <sensor name="imu_sensor">
+      <sensor name="imu">
         <state_interface name="orientation.x"/>
         <state_interface name="orientation.y"/>
